File: hdw/KiCad_Project/Electronic_Calendar/Electronic_Calendar.kicad_pcb (KiCad board)
At the start: 4 copper layers, 432 parts, among them J1501 USB_B_Mini, J201 +12V IN, J601 PICKIT3, Q201 IPC100N04S51R2ATMA1, Q202 IPC100N04S51R2ATMA1, Q401 IPC100N04S51R2ATMA1, Q601 BSS214NW, SW601 MRST, SW901 Cap_Touch, U1001 74LVC1G06, U1002 74LVC1G06, U1003 74LVC1G06, U1004 74LVC1G06, U1005 74LVC1G17, U1006 74LVC1G06, U1101 74LVC1G06, U1102 74LVC1G06, U1103 74LVC1G06, U1104 74LVC1G06, U1105 74LVC1G06, U1106 74LVC1G06, U1401 74HC138, U1402 74HC138, U1403 74HC138, U1404 74HC138, U1405 74HC138, U1501 LT6700-1-S6, U1502 FT234XD, U1503 TPD3S014DBVR, U1601 MCP9804_DFN, U1602 MCP9804_DFN, U1603 MCP9804_DFN, U1604 MCP9804_DFN, U1701 OPA340NA, U1702 OPA340NA, U1703 OPA340NA, U1704 OPA340NA, U1705 OPA340NA, U1706 OPA340NA, U201 LTC4365DDB, U202 INA138, U301 LTC3605A_UF, U302 INA138, U401 LTC4041UFD, U501 74LVC1G17, U502 74LVC1G14, U701 PIC32MZ2048EFG100_IPT, U901 AT42QT1010-TSHR

Commit message: Arranged a few more PCB sections
Parts:
- removed the D1251 at (361.2, 40.6)
- added D1229: Red, LEDs:LED_0603, F.Cu at (408.1, 16.6)
- moved R902 145.1 mm to (130.8, 9.46), turned to 90 degrees
- moved R901 140.7 mm to (130.3, 14.3), turned to 90 degrees
- moved C903 139.3 mm to (133.2, 8.64), turned to 180 degrees
- moved C902 139.2 mm to (133.2, 7.24), turned to 180 degrees
- moved C904 134.6 mm to (133.2, 10.0), turned to 180 degrees
- moved U901 134.5 mm to (133.2, 12.6)
- moved C901 134.3 mm to (133.2, 15.2), turned to 180 degrees
- moved SW901 128.7 mm to (133.2, 20.2), turned to 90 degrees
- moved C1105 104.6 mm to (196.7, 97.7), turned to 180 degrees
- moved U1105 104.5 mm to (196.7, 95.5)
- moved R1109 101.4 mm to (194.2, 96.0), turned to 270 degrees
- moved R1111 98.8 mm to (200.0, 94.7)
- moved D1105 98.7 mm to (200.0, 96.3)
- moved R1105 96.2 mm to (181.7, 94.6), turned to 90 degrees
- moved U1103 93.5 mm to (184.2, 94.1)
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- renumbered D1229 to D1251
Connections:
- C1401 pad 1: +3.3V_SW -> +3V3
- C1402 pad 1: +3.3V_SW -> +3V3
- C1403 pad 1: +3.3V_SW -> +3V3
- C1404 pad 1: +3.3V_SW -> +3V3
- C1405 pad 1: +3.3V_SW -> +3V3
- C1502 pad 1: +3.3V_SW -> +3V3
- C1503 pad 1: +3.3V_SW -> +3V3
- C1701 pad 1: +3.3V_SW -> +3V3
- C1702 pad 1: +3.3V_SW -> +3V3
- C1703 pad 1: +3.3V_SW -> +3V3
- C1704 pad 1: +3.3V_SW -> +3V3
- C1705 pad 1: +3.3V_SW -> +3V3
- C1706 pad 1: +3.3V_SW -> +3V3
- C1709 pad 1: +3.3V_SW -> +3V3
- C1710 pad 1: +3.3V_SW -> +3V3
- C1711 pad 1: +3.3V_SW -> +3V3
- C1712 pad 1: +3.3V_SW -> +3V3
- C1713 pad 1: +3.3V_SW -> +3V3
- C1714 pad 1: +3.3V_SW -> +3V3
- C1717 pad 1: +3.3V_SW -> +3V3
- C1718 pad 1: +3.3V_SW -> +3V3
- C1719 pad 1: +3.3V_SW -> +3V3
- C1720 pad 1: +3.3V_SW -> +3V3
- C1721 pad 1: +3.3V_SW -> +3V3
- C1722 pad 1: +3.3V_SW -> +3V3
- C902 pad 1: +3.3V_SW -> +3V3
- C903 pad 1: +3.3V_SW -> +3V3
- C904 pad 1: +3.3V_SW -> +3V3
- D1251 pad 1: ~MON_LED -> ~SUN_LED
- R1301 pad 1: +3.3V_SW -> +3V3
- R1302 pad 1: +3.3V_SW -> +3V3
- R1303 pad 1: +3.3V_SW -> +3V3
- R1304 pad 1: +3.3V_SW -> +3V3
- R1305 pad 1: +3.3V_SW -> +3V3
- R1306 pad 1: +3.3V_SW -> +3V3
- R1307 pad 1: +3.3V_SW -> +3V3
- R1308 pad 1: +3.3V_SW -> +3V3
- R1309 pad 1: +3.3V_SW -> +3V3
- R1310 pad 1: +3.3V_SW -> +3V3
- R1311 pad 1: +3.3V_SW -> +3V3
- R1312 pad 1: +3.3V_SW -> +3V3
- R1313 pad 1: +3.3V_SW -> +3V3
- R1314 pad 1: +3.3V_SW -> +3V3
- R1315 pad 1: +3.3V_SW -> +3V3
- R1316 pad 1: +3.3V_SW -> +3V3
- R1317 pad 1: +3.3V_SW -> +3V3
- R1318 pad 1: +3.3V_SW -> +3V3
- R1319 pad 1: +3.3V_SW -> +3V3
- R1320 pad 1: +3.3V_SW -> +3V3
- R1321 pad 1: +3.3V_SW -> +3V3
- R1413 pad 1: +3.3V_SW -> +3V3
- R1414 pad 1: +3.3V_SW -> +3V3
- R1423 pad 1: +3.3V_SW -> +3V3
- R1424 pad 1: +3.3V_SW -> +3V3
- R1505 pad 1: +3.3V_SW -> +3V3
- R1506 pad 1: +3.3V_SW -> +3V3
- R1507 pad 1: +3.3V_SW -> +3V3
- R1701 pad 2: +3.3V_SW -> +3V3
- U1401 pad 16: +3.3V_SW -> +3V3
- U1402 pad 16: +3.3V_SW -> +3V3
- U1403 pad 16: +3.3V_SW -> +3V3
- U1404 pad 16: +3.3V_SW -> +3V3
- U1405 pad 16: +3.3V_SW -> +3V3
- U1501 pad 5: +3.3V_SW -> +3V3
- U1502 pad 9: +3.3V_SW -> +3V3
- U1601 pad 7: +3.3V_SW -> +3V3
- U1602 pad 6: +3.3V_SW -> +3V3
- U1604 pad 6: +3.3V_SW -> +3V3
- U1604 pad 7: +3.3V_SW -> +3V3
- U1701 pad 5: +3.3V_SW -> +3V3
- U1702 pad 5: +3.3V_SW -> +3V3
- U1703 pad 5: +3.3V_SW -> +3V3
- U1704 pad 5: +3.3V_SW -> +3V3
- U1705 pad 5: +3.3V_SW -> +3V3
- U1706 pad 5: +3.3V_SW -> +3V3
- U901 pad 5: +3.3V_SW -> +3V3
- U901 pad 6: +3.3V_SW -> +3V3
Other:
- board text added: "1"
- board text added: "10"
- board text added: "11"
- board text added: "12"
- board text added: "13"
- board text added: "14"
- board text added: "15"
- board text added: "16"
- board text added: "17"
- board text added: "18"
- board text added: "19"
- board text added: "2"
- board text added: "20"
- board text added: "2019"
- board text added: "2020"
- board text added: "2021"
- board text added: "2022"
- board text added: "2023"
- board text added: "2024"
- board text added: "2025"
- board text added: "2026"
- board text added: "21"
- board text added: "22"
- board text added: "23"
- board text added: "24"
- board text added: "25"
- board text added: "26"
- board text added: "27"
- board text added: "28"
- board text added: "29"
- board text added: "3"
- board text added: "30"
- board text added: "31"
- board text added: "4"
- board text added: "5"
- board text added: "6"
- board text added: "7"
- board text added: "8"
- board text added: "9"
- board text added: "April"
- board text added: "August"
- board text added: "Calendar"
- board text added: "December"
- board text added: "February"
- board text added: "Friday"
- board text added: "January"
- board text added: "July"
- board text added: "June"
- board text added: "March"
- board text added: "May"
- board text added: "Monday"
- board text added: "November"
- board text added: "October"
- board text added: "STATUS"
- board text added: "Saturday"
- board text added: "September"
- board text added: "Sunday"
- board text added: "Thursday"
- board text added: "Tuesday"
- board text added: "Wednesday"

Commit message: More PCB part placement
Parts:
- removed C1710, C501, C502: 0.1uF, Capacitors_SMD:C_0603
- removed C1712, C1716: 10nF, Capacitors_SMD:C_0603
- removed C1714: 1nF, Capacitors_SMD:C_0603
- removed C405, C406: 47uF, Capacitors_SMD:C_1210
- removed C407: 100uF, Capacitors_Tantalum_SMD:CP_Tantalum_Case-D_EIA-7343-31_Reflow
- removed L401: 2.2uH, Inductors_SMD:L_Vishay_IHLP-2020
- removed Q401: IPC100N04S51R2ATMA1, TO_SOT_Packages_SMD:TDSON-8-1
- removed R1706: 499, Resistors_SMD:R_0603
- removed R407: 121k, Resistors_SMD:R_0603
- removed R408: 75k, Resistors_SMD:R_0603
- removed R409: 12m, Resistors_SMD:R_0805
- removed R410: 0, Resistors_SMD:R_0805
- removed R411: 1k, Resistors_SMD:R_0603
- removed R412: 1.07M, Resistors_SMD:R_0603
- removed R413: 340k, Resistors_SMD:R_0603
- removed R414: 931k, Resistors_SMD:R_0603
- removed R415: 392k, Resistors_SMD:R_0603
- removed TP402: TP, Custom Footprints Library:Test_Point
- removed U1704: OPA340NA, TO_SOT_Packages_SMD:SOT-23-5
- removed U501: 74LVC1G17, TO_SOT_Packages_SMD:SOT-353_SC-70-5
- removed U502: 74LVC1G14, TO_SOT_Packages_SMD:SOT-353_SC-70-5
- added BT401: BR-2/3AE5SPN, Custom Footprints Library:BR-2_3AE5SPN, F.Cu at (196.2, -80.4)
- added TP301: TP, Custom Footprints Library:Test_Point, F.Cu at (159.8, -49.0)
- C401: value 10uF -> 0.1uF; footprint Capacitors_SMD:C_1206 -> Capacitors_SMD:C_0603
- C402: value 2.2nF -> 47uF; footprint Capacitors_SMD:C_0603 -> Capacitors_SMD:C_1210
- C403: value 10uF -> 47uF; footprint Capacitors_SMD:C_1206 -> Capacitors_SMD:C_1210
- C404: value 10F -> 47uF; footprint Custom Footprints Library:SCCS30B106PRB -> Capacitors_SMD:C_1210
- R1301, R1302, R1303, R1304, R1305, R1306, R1307, R1308, R1309, R1310, R1311, R1312, R1313, R1314, R1315, R1316, R1317, R1318, R1319, R1320, R1321: moved to B.Cu
- R401, R402: value 2M -> 243k
- R403, R406: value 2M -> 10k
- R404, R405: value 2M -> 499
- U401: value LTC4041UFD -> LTC4415DHC; footprint Housings_DFN_QFN:QFN-24-1EP_4x5mm_Pitch0.5mm -> Housings_DFN_QFN:DFN-16-1EP_3x5mm_Pitch0.5mm
- moved D1309 381.2 mm to (541.9, 34.0)
- moved D1311 380.3 mm to (541.9, 39.1)
- moved D1320 377.8 mm to (536.8, 39.1)
- moved D1310 375.9 mm to (541.9, 36.5)
- moved D1312 375.0 mm to (541.9, 41.6)
- moved D1321 371.7 mm to (536.8, 41.6)
- moved R1309 370.7 mm to (541.9, 34.0)
- moved R1312 370.4 mm to (541.9, 41.6)
- moved D1306 370.0 mm to (531.7, 36.5)
- moved R1305 366.8 mm to (531.7, 34.0)
- moved D1318 366.6 mm to (526.7, 41.6)
- moved C209 366.4 mm to (433.3, 164.0), turned to 90 degrees
- moved D1308 366.1 mm to (531.7, 41.6)
- moved R1310 365.7 mm to (541.9, 36.5)
- moved D1319 363.6 mm to (536.8, 36.5)
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Connections:
- C401 pad 1: +3V3 -> VBAT_ADC
- C402 pad 1: Net-(C402-Pad1) -> +3.3V_SW
- C403 pad 1: +3.3V_BCKP -> VBAT
- C404 pad 1: VTANK -> +3.3V_BCKP
- R401 pad 1: +3.3V_BCKP -> VBAT
- R401 pad 2: ~BCKP_PFO -> VBAT_ADC
- R402 pad 1: +3.3V_BCKP -> VBAT_ADC
- R402 pad 2: BCKP_SYSGD -> GND
- R403 pad 1: +3.3V_BCKP -> VBAT_ADC
- R403 pad 2: BCKP_CAPGD -> GND
- R404 pad 1: +3.3V_BCKP -> Net-(R404-Pad1)
- R404 pad 2: ~BCKP_CHGEN -> GND
- R405 pad 1: +3.3V_BCKP -> Net-(R405-Pad1)
- R405 pad 2: ~BCKP_CAPFLT -> GND
- R406 pad 1: +3.3V_BCKP -> +3V3
- R406 pad 2: ~BCKP_BSTEN -> ~DIODE_FAULT
- U1002 pad 2: BCKP_SYSGD -> (no net)
- U1004 pad 2: BCKP_CAPGD -> (no net)
- U1005 pad 2: ~BCKP_CAPFLT -> ~DIODE_FAULT
- U401 pad 1: +3.3V_BCKP -> +3.3V_SW
- U401 pad 10: Net-(R412-Pad2) -> +3.3V_BCKP
- U401 pad 11: BCKP_SYSGD -> (no net)
- U401 pad 12: Net-(R414-Pad2) -> ~DIODE_FAULT
- U401 pad 13: BCKP_CAPGD -> ~DIODE_FAULT
- U401 pad 14: ~BCKP_PFO -> (no net)
- U401 pad 15: Net-(Q401-Pad4) -> +3.3V_BCKP
- U401 pad 16: +3V3 -> +3.3V_BCKP
- U401 pad 17: Net-(C402-Pad1) -> GND
- U401 pad 2: Net-(R411-Pad1) -> +3.3V_SW
- U401 pad 3: BCKP_IMON -> POS3P3_PGOOD
- U401 pad 4: ~BCKP_CHGEN -> Net-(R404-Pad1)
- U401 pad 5: ~BCKP_BSTEN -> Net-(R405-Pad1)
- U401 pad 6: +3V3 -> POS3P3_PGOOD
- U401 pad 7: Net-(Q401-Pad1) -> VBAT
- U401 pad 8: ~BCKP_CAPFLT -> VBAT
- U401 pad 9: (no net) -> +3.3V_BCKP
- U701 pad 11: POS3P3_PGOOD -> POS12_PGOOD
- U701 pad 12: POS3P3_PGOOD -> POS12_PGOOD
- U701 pad 28: (no net) -> VBAT_ADC
- U701 pad 39: ~BCKP_CAPFLT -> ~DIODE_FAULT
- U701 pad 40: BCKP_CAPGD -> (no net)
- U701 pad 50: POS12_PGOOD -> POS3P3_PGOOD
- U701 pad 58: BCKP_SYSGD -> (no net)
- U701 pad 61: BCKP_IMON_ADC -> (no net)
- U701 pad 65: ~BCKP_PFO -> (no net)
Other:
- board text added: "+12VIN"
- board text added: "Analog"
- board text added: "Clock"
- board text added: "Hours"
- board text added: "INPUT"
- board text added: "Minutes"
- board text added: "Seconds"

Commit message: More part arranging on PCB
Parts:
- removed C303: 22uF, Capacitors_SMD:C_2220
- added C825: 0.1uF, Capacitors_SMD:C_0603, F.Cu at (211.5, 108.9)
- added Q401: 2N7002, TO_SOT_Packages_SMD:SOT-23, F.Cu at (572.1, 165.0)
- added R407: 243k, Resistors_SMD:R_0603, F.Cu at (558.4, 160.5)
- added R801: 10k, Resistors_SMD:R_0603, F.Cu at (208.8, 112.1)
- added TP402: TP, Custom Footprints Library:Test_Point, F.Cu at (558.0, 168.0)
- added U402: TPS22929D, TO_SOT_Packages_SMD:SOT-23-6, F.Cu at (558.4, 163.6)
- added U801: TPS22929D, TO_SOT_Packages_SMD:SOT-23-6, F.Cu at (208.8, 109.3)
- moved TP401 470.0 mm to (574.0, 155.8)
- moved U401 448.7 mm to (566.4, 159.7)
- moved C401 448.1 mm to (568.7, 164.0)
- moved R403 446.8 mm to (572.1, 162.4), turned to 180 degrees
- moved C403 443.4 mm to (562.2, 163.8), turned to 270 degrees
- moved R402 442.7 mm to (568.7, 165.7)
- moved R404 432.7 mm to (561.4, 159.0), turned to 180 degrees
- moved R405 430.5 mm to (561.4, 160.5), turned to 180 degrees
- moved C404 429.6 mm to (572.1, 159.7)
- moved R401 427.1 mm to (565.9, 165.7)
- moved R406 424.2 mm to (569.5, 155.8), turned to 270 degrees
- moved C402 421.6 mm to (562.2, 155.8), turned to 90 degrees
- moved BT401 416.4 mm to (536.6, 159.3)
- moved TP301 68.6 mm to (201.4, 5.46)
Connections:
- net ~USB_ACTIVE renamed ~USB_TRAFFIC
- BT401 pad 1: VBAT -> Net-(BT401-Pad1)
- C402 pad 1: +3.3V_SW -> +3V3
- R1001 pad 1: +3V3 -> +3.3V_STAT
- R1003 pad 1: +3V3 -> +3.3V_STAT
- R1005 pad 1: +3V3 -> +3.3V_STAT
- R1006 pad 1: +3V3 -> +3.3V_STAT
- R1103 pad 1: +3V3 -> +3.3V_STAT
- R1104 pad 1: +3V3 -> +3.3V_STAT
- R1107 pad 1: +3V3 -> +3.3V_STAT
- R1108 pad 1: +3V3 -> +3.3V_STAT
- R1111 pad 1: +3V3 -> +3.3V_STAT
- R1112 pad 1: +3V3 -> +3.3V_STAT
- R402 pad 2: GND -> Net-(Q401-Pad3)
- R403 pad 1: VBAT_ADC -> VBAT_ADC_EN
- U401 pad 1: +3.3V_SW -> +3V3
- U401 pad 2: +3.3V_SW -> +3V3
- U701 pad 40: (no net) -> VBAT_ADC_EN
- U701 pad 58: (no net) -> STATUS_LED_ENABLE
- U701 pad 65: (no net) -> ~VBAT_ISOLATE
Other:
- board text added: "+3.3V BCKP"
- board text added: "Backup"
- board text added: "VBAT"

Commit message: even more arranging
Parts:
- removed R1601, R1602, R1603, R1604, R1605, R1606, R1613, R1614: 100, Resistors_SMD:R_0603
- moved C1610 622.7 mm to (657.2, 43.2), turned to 180 degrees
- moved U1604 618.2 mm to (656.5, 48.7)
- moved U1603 617.0 mm to (648.2, 48.7)
- moved C1612 615.1 mm to (657.2, 46.1), turned to 180 degrees
- moved C1611 613.5 mm to (657.2, 44.6), turned to 180 degrees
- moved R1615 612.4 mm to (654.9, 45.5), turned to 270 degrees
- moved R1616 610.1 mm to (653.3, 45.5), turned to 270 degrees
- moved U1602 607.6 mm to (639.5, 48.7)
- moved C1603 607.0 mm to (648.9, 43.2), turned to 180 degrees
- moved C1608 604.9 mm to (640.2, 46.1), turned to 180 degrees
- moved C1605 604.8 mm to (640.2, 44.6), turned to 180 degrees
- moved C1606 603.0 mm to (648.9, 44.6), turned to 180 degrees
- moved C1602 601.3 mm to (640.2, 43.2), turned to 180 degrees
- moved U1601 599.0 mm to (631.6, 48.7)
- moved C1609 598.9 mm to (648.9, 46.1), turned to 180 degrees
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Connections:
- R1607 pad 2: Net-(R1601-Pad2) -> TEMP_I2C_SDA
- R1608 pad 2: Net-(R1603-Pad2) -> TEMP_I2C_SDA
- R1609 pad 2: Net-(R1605-Pad2) -> TEMP_I2C_SDA
- R1610 pad 2: Net-(R1602-Pad2) -> TEMP_I2C_SCL
- R1611 pad 2: Net-(R1604-Pad2) -> TEMP_I2C_SCL
- R1612 pad 2: Net-(R1606-Pad2) -> TEMP_I2C_SCL
- R1615 pad 2: Net-(R1613-Pad2) -> TEMP_I2C_SDA
- R1616 pad 2: Net-(R1614-Pad2) -> TEMP_I2C_SCL
- U1601 pad 1: Net-(R1601-Pad2) -> TEMP_I2C_SDA
- U1601 pad 2: Net-(R1602-Pad2) -> TEMP_I2C_SCL
- U1602 pad 1: Net-(R1603-Pad2) -> TEMP_I2C_SDA
- U1602 pad 2: Net-(R1604-Pad2) -> TEMP_I2C_SCL
- U1603 pad 1: Net-(R1605-Pad2) -> TEMP_I2C_SDA
- U1603 pad 2: Net-(R1606-Pad2) -> TEMP_I2C_SCL
- U1604 pad 1: Net-(R1613-Pad2) -> TEMP_I2C_SDA
- U1604 pad 2: Net-(R1614-Pad2) -> TEMP_I2C_SCL
Other:
- board text added: "+12V"
- board text added: "Power"
- board text added: "Temp"

Commit message: Finished grouping parts on PCB
Parts:
- removed C1002, C1004: 0.1uF, Capacitors_SMD:C_0603
- removed D1002, D1004: Green, LEDs:LED_0603
- removed R1002, R1004: 1k, Resistors_SMD:R_0603
- removed U1002, U1004: 74LVC1G06, TO_SOT_Packages_SMD:SOT-353_SC-70-5
- C1501, C1502, C1503, C1504, C1505, C1506, C1507, C1508, C1509, C1510, D1501, L1501, L1502, R1501, R1502, R1503, R1504, R1505, R1506, R1507, R1508, R1509, R1510, TP1501, U1501, U1502, U1503: moved to B.Cu
- moved R1001 344.9 mm to (-74.2, 175.8)
- moved D1001 342.4 mm to (-74.2, 177.2)
- moved U1001 342.0 mm to (-77.9, 176.5)
- moved C1001 341.0 mm to (-77.9, 178.8), turned to 180 degrees
- moved R1003 334.4 mm to (-59.6, 175.8)
- moved C1003 330.6 mm to (-63.2, 178.8), turned to 180 degrees
- moved D1003 323.5 mm to (-59.6, 177.2)
- moved C1005 322.9 mm to (-50.7, 178.8), turned to 180 degrees
- moved R1005 321.5 mm to (-47.1, 175.8)
- moved U1003 318.4 mm to (-63.2, 176.5)
- moved R1006 311.7 mm to (-37.5, 175.8)
- moved U1005 310.7 mm to (-50.7, 176.5)
- moved D1005 310.4 mm to (-47.1, 177.2)
- moved C1006 308.1 mm to (-41.0, 178.8), turned to 180 degrees
- moved D1006 296.7 mm to (-37.5, 177.2)
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Other:
- board text added: "+3.3V"
- board text added: "+5V USB"
- board text added: "Buck"
- board text added: "Driver"
- board text added: "PGOOD"
- board text added: "USB"
- board text added: "USB Traffic"

Commit message: Decided on shape and placed sections onto PCB
Parts:
- removed TP1502, TP202: TP, Pin_Headers:Pin_Header_Angled_1x01_Pitch2.54mm
- C1501, C1502, C1503, C1504, C1505, C1506, C1507, C1508, C1509, C1510, D1501, L1501, L1502, R1301, R1302, R1303, R1304, R1305, R1306, R1307, R1308, R1309, R1310, R1311, R1312, R1313, R1314, R1315, R1316, R1317, R1318, R1319, R1320, R1321, R1501, R1502, R1503, R1504, R1505, R1506, R1507, R1508, R1509, R1510, TP1501, U1501, U1502, U1503: moved to F.Cu
- D1201, D1202, D1203, D1204, D1205, D1206, D1207, D1208, D1209, D1210, D1211, D1212, D1213, D1214, D1215, D1216, D1217, D1218, D1219, D1220, D1221, D1222, D1223, D1224, D1225, D1226, D1227, D1228, D1229, D1230, D1231, D1232, D1233, D1234, D1235, D1236, D1237, D1238, D1239, D1240, D1241, D1242, D1243, D1244, D1245, D1246, D1247, D1248, D1249, D1250, D1251, D1252, D1253, D1254, D1255, D1256, D1257, D1258, D1301, D1302, D1303, D1304, D1305, D1306, D1307, D1308, D1309, D1310, D1311, D1312, D1313, D1314, D1315, D1316, D1317, D1318, D1319, D1320, D1321, J1501, J201, SW901: moved to B.Cu
- moved SW901 339.1 mm to (73.4, 138.9), turned to 270 degrees
- moved C901 339.0 mm to (73.4, 143.0)
- moved C902 339.0 mm to (73.4, 135.0)
- moved C903 339.0 mm to (73.4, 136.4)
- moved C904 339.0 mm to (73.4, 137.8)
- moved R901 339.0 mm to (70.5, 142.0)
- moved U901 339.0 mm to (73.4, 140.4)
- moved R902 339.0 mm to (71.1, 137.2)
- moved R1608 320.9 mm to (83.7, 137.3)
- moved C1602 320.9 mm to (86.1, 135.0)
- moved C1605 320.9 mm to (86.1, 136.5)
- moved C1608 320.9 mm to (86.1, 137.9)
- moved R1611 320.9 mm to (82.2, 137.3)
- moved U1602 320.9 mm to (85.4, 140.5)
- moved U1603 309.2 mm to (93.4, 48.2), turned to 270 degrees
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Other:
- board outline added: 100 x 100 mm
- board text added: "+12V PGOOD"
- board text added: "+3.3V PGOOD"
- board text added: "+5V USB PGOOD"
- board text added: "Analog Error"
- board text added: "CPU Exception"
- board text added: "Diode Fault"
- board text added: "Heart Beat"
- board text added: "Other Error"
- board text added: "Reset/ Prog"
- board text added: "USB Error"
- board text removed: "Analog"
- board text removed: "Backup"
- board text removed: "Buck"
- board text removed: "Calendar"
- board text removed: "Clock"
- board text removed: "Driver"
- board text removed: "INPUT"
- board text removed: "MCU"
- board text removed: "PGOOD"
- board text removed: "Power"
- board text removed: "STATUS"
- board text removed: "Temp"
- board text removed: "USB"

Commit message: Began routing
Parts:
- moved TP201 24.3 mm to (91.6, 142.1), turned to 0 degrees
- moved U901 10.5 mm to (73.3, 129.9)
- moved C902 10.5 mm to (73.3, 124.5)
- moved C901 10.5 mm to (73.3, 132.5)
- moved C903 10.5 mm to (73.3, 125.9)
- moved R901 10.5 mm to (70.5, 131.5)
- moved R902 10.5 mm to (71.0, 126.7)
- moved C904 10.5 mm to (73.3, 127.3)
Routing:
- net Net-(D1213-Pad2): track 0.00 -> 77.7 mm, vias 0 -> 1
- net Net-(D1201-Pad2): track 0.00 -> 29.5 mm, vias 0 -> 1
- net Date_Decode_Enable: track 0.00 -> 27.4 mm
- net GND: track 0.00 -> 25.8 mm, vias 0 -> 8
- net Date_B2: track 0.00 -> 20.6 mm
- net Date_B0: track 0.00 -> 20.3 mm
- net Net-(D1232-Pad2): track 0.00 -> 19.3 mm, vias 0 -> 1
- net Date_B1: track 0.00 -> 19.1 mm
- net Net-(D1229-Pad2): track 0.00 -> 16.8 mm, vias 0 -> 1
- net +3V3: track 0.00 -> 14.3 mm
- net Net-(R901-Pad1): track 0.00 -> 9.34 mm, vias 0 -> 1
- net ~Date_Decode_2: track 0.00 -> 5.24 mm
- net ~Date_Decode_1: track 0.00 -> 5.24 mm
- net ~Date_Decode_4: track 0.00 -> 5.24 mm
- net ~Date_Decode_3: track 0.00 -> 5.24 mm
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- added copper zone on GND, net GND
Other:
- board text added: "Power"

Commit message: More routing
Parts:
- moved R1202 0.77 mm to (110.0, 141.9)
- moved D1255 0.76 mm to (94.9, 68.3)
Routing:
- net GND: track 25.8 -> 208.9 mm, vias 8 -> 73
- net +3V3: track 14.3 -> 116.7 mm, vias 0 -> 2
- net ~Date27_LED: track 0.00 -> 60.0 mm, vias 0 -> 1
- net ~Date24_LED: track 0.00 -> 57.6 mm, vias 0 -> 1
- net ~Date26_LED: track 0.00 -> 57.6 mm, vias 0 -> 1
- net ~Date25_LED: track 0.00 -> 55.2 mm, vias 0 -> 1
- net ~Date28_LED: track 0.00 -> 49.1 mm, vias 0 -> 1
- net ~Date29_LED: track 0.00 -> 48.0 mm, vias 0 -> 1
- net ~Date31_LED: track 0.00 -> 47.6 mm, vias 0 -> 1
- net ~Date30_LED: track 0.00 -> 46.9 mm, vias 0 -> 1
- net +3.3V_BCKP: track 0.00 -> 46.4 mm
- net ~Date23_LED: track 0.00 -> 45.4 mm, vias 0 -> 1
- net ~Date22_LED: track 0.00 -> 42.9 mm, vias 0 -> 1
- net ~Date21_LED: track 0.00 -> 40.3 mm, vias 0 -> 1
- net ~Date1_LED: track 0.00 -> 39.4 mm, vias 0 -> 2
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