File: hdw/KiCad_Project/Electronic_Calendar/Electronic_Calendar.kicad_pcb (KiCad board)
At the start: 4 copper layers, 100 x 100 mm, 397 parts, among them J1501 USB_B_Mini, J201 +12V IN, J601 PICKIT3, Q201 IPC100N04S51R2ATMA1, Q202 IPC100N04S51R2ATMA1, Q401 2N7002, Q601 BSS214NW, SW601 MRST, SW901 Cap_Touch, U1001 74LVC1G06, U1003 74LVC1G06, U1005 74LVC1G17, U1006 74LVC1G06, U1101 74LVC1G06, U1102 74LVC1G06, U1103 74LVC1G06, U1104 74LVC1G06, U1105 74LVC1G06, U1106 74LVC1G06, U1401 74HC138, U1402 74HC138, U1403 74HC138, U1404 74HC138, U1405 74HC138, U1501 LT6700-1-S6, U1502 FT234XD, U1503 TPD3S014DBVR, U1601 MCP9804_DFN, U1602 MCP9804_DFN, U1603 MCP9804_DFN, U1604 MCP9804_DFN, U1701 OPA340NA, U1702 OPA340NA, U1703 OPA340NA, U1705 OPA340NA, U1706 OPA340NA, U201 LTC4365DDB, U202 INA138, U301 LTC3605A_UF, U302 INA138, U401 LTC4415DHC, U402 TPS22929D, U701 PIC32MZ2048EFG100_IPT, U801 TPS22929D, U901 AT42QT1010-TSHR

Commit message: Way more routing
Parts:
- moved R601 30.0 mm to (150.6, 131.1), turned to 90 degrees
- moved R602 27.9 mm to (152.1, 131.1), turned to 270 degrees
- moved Q601 24.7 mm to (154.7, 131.1), turned to 0 degrees
- moved C602 24.6 mm to (153.7, 128.8), turned to 180 degrees
- moved R603 21.5 mm to (157.4, 131.1), turned to 270 degrees
- moved R605 20.9 mm to (156.6, 128.8), turned to 180 degrees
- moved R604 20.0 mm to (156.6, 127.2), turned to 0 degrees
- moved TP301 18.2 mm to (129.5, 46.9)
- moved R606 17.6 mm to (158.8, 128.0), turned to 270 degrees
- moved C205 1.02 mm to (97.5, 66.2)
- moved C206 1.02 mm to (97.5, 64.7)
- moved C207 1.02 mm to (97.5, 63.2)
- moved C208 1.02 mm to (102.0, 59.2)
- moved R210 1.02 mm to (100.5, 59.2)
- moved U202 1.02 mm to (97.7, 58.7)
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Connections:
- U701 pad 1: ~Date_Decode_2 -> ~Minutes1_LED
- U701 pad 100: ~THR_LED -> ~Minutes6_LED
- U701 pad 2: POS3P3_ADC -> ~Minutes3_LED
- U701 pad 20: ~Hours3_LED -> (no net)
- U701 pad 21: ~Hours2_LED -> ~Hours1_LED
- U701 pad 22: ~Hours1_LED -> ~Hours3_LED
- U701 pad 23: ~Hours0_LED -> ~Hours5_LED
- U701 pad 26: ~Hours4_LED -> (no net)
- U701 pad 27: ~Hours5_LED -> (no net)
- U701 pad 3: ~FRI_LED -> ~Minutes5_LED
- U701 pad 32: ~Hours6_LED -> (no net)
- U701 pad 33: ~Minutes0_LED -> (no net)
- U701 pad 34: ~Minutes1_LED -> (no net)
- U701 pad 35: ~Minutes2_LED -> (no net)
- U701 pad 4: ~SAT_LED -> (no net)
- U701 pad 41: ~Minutes3_LED -> (no net)
- U701 pad 42: ~Minutes4_LED -> (no net)
- U701 pad 43: ~Minutes5_LED -> (no net)
- U701 pad 44: ~Minutes6_LED -> (no net)
- U701 pad 47: ~DEC_LED -> (no net)
- U701 pad 49: ~Seconds4_LED -> (no net)
- U701 pad 50: POS3P3_PGOOD -> ~SUN_LED
- U701 pad 56: Analog_Error_LED -> ~MON_LED
- U701 pad 57: Other_Error_LED -> ~TUE_LED
- U701 pad 58: STATUS_LED_ENABLE -> ~WED_LED
- U701 pad 59: POS12_ISNS_ADC -> ~THR_LED
- U701 pad 6: ~Seconds0_LED -> ~Hours0_LED
- U701 pad 60: POS5_USB_ADC -> ~FRI_LED
- U701 pad 61: (no net) -> ~SAT_LED
- U701 pad 7: ~Seconds1_LED -> ~Hours2_LED
- U701 pad 72: ~Seconds5_LED -> (no net)
- U701 pad 73: ~Seconds6_LED -> (no net)
- U701 pad 79: ~OCT_LED -> ~MAY_LED
- U701 pad 8: ~Seconds2_LED -> ~Hours4_LED
- U701 pad 80: ~NOV_LED -> ~JUN_LED
- U701 pad 81: ~MAY_LED -> ~OCT_LED
- U701 pad 82: ~JUN_LED -> ~NOV_LED
- U701 pad 85: Heartbeat_LED -> ~DEC_LED
- U701 pad 86: USB_Error_LED -> ~Seconds0_LED
- U701 pad 89: ~Date_Decode_3 -> ~Seconds2_LED
- U701 pad 9: ~Seconds3_LED -> ~Hours6_LED
- U701 pad 90: ~Date_Decode_4 -> ~Seconds4_LED
- U701 pad 91: ~SUN_LED -> ~Seconds6_LED
- U701 pad 94: ~MON_LED -> ~Seconds1_LED
- U701 pad 95: ~Date_Decode_1 -> ~Seconds3_LED
- U701 pad 96: Date_B1 -> ~Seconds5_LED
- U701 pad 97: Date_B2 -> ~Minutes0_LED
- U701 pad 98: ~TUE_LED -> ~Minutes2_LED
- U701 pad 99: ~WED_LED -> ~Minutes4_LED
Routing:
- net ~JAN_LED: track 0.00 -> 123.5 mm, vias 0 -> 2
- net GND: track 208.9 -> 326.2 mm, vias 73 -> 157
- net +3V3: track 116.7 -> 231.0 mm, vias 2 -> 154
- net +3.3V_STAT: track 0.00 -> 100.4 mm
- net ~SEP_LED: track 0.00 -> 92.8 mm, vias 0 -> 1
- net ~JUL_LED: track 0.00 -> 92.6 mm, vias 0 -> 1
- net ~AUG_LED: track 0.00 -> 92.2 mm, vias 0 -> 1
- net ~SAT_LED: track 0.00 -> 80.8 mm, vias 0 -> 1
- net ~FRI_LED: track 0.00 -> 79.6 mm, vias 0 -> 1
- net ~THR_LED: track 0.00 -> 78.9 mm, vias 0 -> 1
- net ~WED_LED: track 0.00 -> 78.2 mm, vias 0 -> 1
- net ~TUE_LED: track 0.00 -> 77.4 mm, vias 0 -> 1
- net ~MON_LED: track 0.00 -> 76.9 mm, vias 0 -> 1
- net ~SUN_LED: track 0.00 -> 76.1 mm, vias 0 -> 1
- net +5V_USB: track 0.00 -> 60.1 mm
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- added copper zone on F.Cu, net +12V
- added copper zone on F.Cu, net +12Vin
- added copper zone on F.Cu, net +3.3V_BCKP
- added copper zone on PWR, net +3.3V_BCKP
- added copper zone on F.Cu, net +3V3
- added copper zone on PWR, net +3V3
- added copper zone on F.Cu, net Net-(BT401-Pad1)
- added copper zone on F.Cu, net Net-(C307-Pad2)
- added copper zone on F.Cu, net Net-(C312-Pad1)
- added copper zone on F.Cu, net Net-(J1501-Pad1)
- added copper zone on F.Cu, net Net-(Q201-Pad1)
- added copper zone on F.Cu, net Net-(Q202-Pad5)
- added copper zone on F.Cu, net VBAT

Commit message: Even more routing
Connections:
- U701 pad 16: Date_B0 -> Date_B1
- U701 pad 17: POS12_ADC -> Date_B0
- U701 pad 4: (no net) -> ~Date_Decode_4
- U701 pad 47: (no net) -> USB_UART_TX
- U701 pad 48: Reset_LED -> USB_UART_RX
- U701 pad 5: Year_B0 -> Date_B2
- U701 pad 87: USB_UART_TX -> Other_Error_LED
- U701 pad 88: USB_UART_RX -> USB_Error_LED
Routing:
- net Date_B2: track 20.6 -> 168.6 mm, vias 0 -> 5
- net Date_B0: track 20.3 -> 162.2 mm, vias 0 -> 7
- net Date_B1: track 19.1 -> 159.4 mm, vias 0 -> 7
- net ~Date_Decode_4: track 5.24 -> 116.1 mm
- net Cap_Touch_Power: track 2.38 -> 111.3 mm, vias 0 -> 2
- net USB_UART_RX: track 2.34 -> 87.3 mm
- net USB_Error_LED: track 1.56 -> 86.1 mm, vias 0 -> 2
- net Other_Error_LED: track 1.55 -> 82.2 mm, vias 0 -> 2
- net USB_UART_TX: track 2.48 -> 83.1 mm
- net GND: track 326.2 -> 341.6 mm
- net +3V3: track 231.0 -> 237.7 mm
- net POS12_PGOOD: track 6.96 -> 7.46 mm

Commit message: More routing
Parts:
- added D1601: MBR0530, Diodes_SMD:D_SOD-123, F.Cu at (120.2, 83.4)
- added D1602: MBR0530, Diodes_SMD:D_SOD-123, F.Cu at (121.5, 103.8)
- added REF**: Keystone_1058_1x2032-CoinCell, Battery_Holders:Keystone_1058_1x2032-CoinCell, F.Cu at (157.1, 82.5)
Connections:
- R1703 pad 2: Net-(R1703-Pad2) -> Net-(D1601-Pad1)
- R1705 pad 2: Net-(R1705-Pad2) -> Net-(D1602-Pad1)
- U1701 pad 1: Net-(R1703-Pad2) -> Net-(D1601-Pad2)
- U1701 pad 4: Net-(R1703-Pad2) -> Net-(D1601-Pad1)
- U1703 pad 1: Net-(R1705-Pad2) -> Net-(D1602-Pad2)
- U1703 pad 4: Net-(R1705-Pad2) -> Net-(D1602-Pad1)
- U701 pad 20: (no net) -> Year_B0
- U701 pad 28: VBAT_ADC -> (no net)
- U701 pad 41: (no net) -> ~Date_Decode_1
- U701 pad 42: (no net) -> ~Date_Decode_2
- U701 pad 43: (no net) -> ~Date_Decode_3
- U701 pad 44: (no net) -> VBAT_ADC
Routing:
- net Year_B0: track 5.07 -> 169.8 mm, vias 0 -> 2
- net Year_B2: track 5.15 -> 161.6 mm, vias 0 -> 4
- net Year_B1: track 4.79 -> 159.5 mm, vias 0 -> 4
- net Date_Decode_Enable: track 27.4 -> 167.4 mm, vias 0 -> 8
- net ~Date_Decode_1: track 5.24 -> 133.8 mm, vias 0 -> 4
- net ~Date_Decode_2: track 5.24 -> 124.6 mm, vias 0 -> 4
- net ~Date_Decode_3: track 5.24 -> 115.1 mm, vias 0 -> 4
- net ~DIODE_FAULT: track 6.98 -> 95.9 mm, vias 2 -> 6
- net VBAT_ADC_EN: track 1.75 -> 78.6 mm, vias 0 -> 4
- net VBAT_ADC: track 2.95 -> 73.8 mm, vias 0 -> 2
- net +3.3V_STAT: track 100.4 -> 159.0 mm, vias 0 -> 2
- net Exception_LED: track 1.56 -> 58.0 mm, vias 0 -> 2
- net POS3P3_ISNS_ADC: track 1.65 -> 46.0 mm, vias 0 -> 2
- net POS5_USB_PGOOD: track 10.0 -> 43.8 mm, vias 0 -> 2
- net ~VBAT_ISOLATE: track 2.03 -> 20.5 mm, vias 0 -> 2
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
Commit message: Finished routing
Parts:
- added G***: Owl_1_Logo, Custom Footprints Library:Owl_1_Logo, F.Cu at (85.0, 127.5)
- added G***: PIC32_Logo, Custom Footprints Library:PIC32_Logo, F.Cu at (135.2, 126.4)
- added REF**: MountingHole_3mm, Mounting_Holes:MountingHole_3mm, F.Cu at (70.6, 62.2)
- added REF**: MountingHole_3mm, Mounting_Holes:MountingHole_3mm, F.Cu at (164.0, 62.2)
Connections:
- U701 pad 26: (no net) -> POS5_USB_ADC
- U701 pad 27: (no net) -> POS12_ADC
- U701 pad 28: (no net) -> Reset_LED
- U701 pad 32: (no net) -> POS3P3_ADC
- U701 pad 33: (no net) -> POS12_ISNS_ADC
- U701 pad 34: (no net) -> Analog_Error_LED
- U701 pad 35: (no net) -> STATUS_LED_ENABLE
- U701 pad 49: (no net) -> Heartbeat_LED
- U701 pad 72: (no net) -> POS3P3_PGOOD
- U701 pad 73: (no net) -> POS5_USB_PGOOD
Routing:
- net TEMP_I2C_SCL: track 32.5 -> 292.4 mm, vias 2 -> 11
- net TEMP_I2C_SDA: track 20.7 -> 269.9 mm, vias 2 -> 11
- net POS12_PGOOD: track 7.46 -> 173.3 mm, vias 0 -> 8
- net +5V_USB: track 60.1 -> 166.5 mm, vias 0 -> 2
- net POS3P3_ISNS: track 3.32 -> 82.5 mm, vias 0 -> 10
- net POS3P3_PGOOD: track 28.6 -> 105.3 mm, vias 2 -> 4
- net STATUS_LED_ENABLE: track 1.93 -> 75.0 mm, vias 0 -> 4
- net Heartbeat_LED: track 1.56 -> 71.3 mm, vias 0 -> 4
- net Reset_LED: track 1.56 -> 71.2 mm, vias 0 -> 6
- net POS12_ISNS_ADC: track 1.65 -> 67.0 mm, vias 0 -> 2
- net Analog_Error_LED: track 1.56 -> 66.4 mm, vias 0 -> 3
- net POS3P3_ADC: track 1.65 -> 56.6 mm, vias 0 -> 2
- net +12V: track 39.4 -> 86.5 mm, vias 2 -> 4
- net POS5_USB_ADC: track 1.65 -> 48.6 mm, vias 0 -> 2
- net POS5_USB_PGOOD: track 43.8 -> 90.5 mm, vias 2 -> 4
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- added copper zone on F.Cu, net GND
Other:
- board text added: "Binary Clock"
- board text added: "Date"
- board text added: "Day"
- board text added: "MRST"
- board text added: "Month"
- board text added: "Printed Circuit Calendar"
- board text added: "Year"

Commit message: Updated PDF, BOM, Gerbers
Parts:
- added G***: Microchip_Logo, Custom Footprints Library:Microchip_Logo, F.Cu at (144.2, 115.5)
- added REF**: KiCAD Logo, Symbols:Symbol_KiCAD-Logo_CopperAndSilkScreenTop, F.Cu at (87.8, 129.5)
- added REF**: Symbol_Barrel_Polarity, Symbols:Symbol_Barrel_Polarity, B.Cu at (81.5, 47.0)
- added REF***: ESD-Logo_6.6x6mm_SilkScreen, Symbols:ESD-Logo_6.6x6mm_SilkScreen, F.Cu at (162.6, 113.5)
- moved G*** 51.7 mm to (103.9, 79.4)
Routing:
- net Net-(C307-Pad2): track 3.36 -> 6.18 mm
Other:
- board text added: "+"
- board text added: "-"
- board text added: "GND"
- board text added: "PICKIT 3"
- board text added: "USB COM Port: 115.2 kbps 8 bit data length No parity 1 stop bit No flow control"
